Commit message: Revised solidworks model
Now includes IMU and LiDAR

File: urdf/arm.urdf.xacro (robot description, xacro)
@@ -6,5 +6,5 @@
     <!-- Included URDF Files -->
     <!--<include filename="$(find turtlebot_description)/urdf/turtlebot.urdf.xacro" />-->
-    <include filename="$(find turtlebot_arm_description)/urdf/arm.xacro" />
+    <include filename="$(find jr_description)/urdf/arm.xacro" />
     <!-- For now I have removed the turtlebot since this all moved around..
     <turtlebot />-->

File: urdf/arm.xacro (robot description, xacro)
@@ -1,5 +1,5 @@
 <?xml version="1.0"?>
 <robot>
-  <include filename="$(find turtlebot_arm_description)/urdf/arm_hardware.xacro" />
+  <include filename="$(find jr_description)/urdf/arm_hardware.xacro" />
   <material name="white">
     <color rgba="0.87 0.90 0.87 1.0"/>

File: urdf/jr.urdf.xacro (robot description, xacro)
@@ -1,3 +1,15 @@
 <?xml version="1.0"?>
-<robot>
+<robot name="jr">
+  <link name="base_footprint" />
+  <joint name="base_footprint_to_base_link" type="fixed">
+    <parent link="base_footprint" />
+    <child link="base_link" />
+    <origin xyz="0 0 0.0587375" rpy="0 0 0"/>
+    <axis xyz="0 0 0" />
+  </joint>
+  <include filename="$(find jr_description)/urdf/jr_description.urdf" />
+  <include filename="$(find jr_description)/urdf/arm.xacro" />
+  <turtlebot_arm parent="arm_base" color="white" gripper_color="green">
+    <origin xyz="0 0 ${AX12_WIDTH/2}"/>
+  </turtlebot_arm>
 </robot>

File: urdf/jr_description.urdf (robot description, URDF)
Before this commit: robot jr_description, 7 links, 6 joints
Links:
- added link imu, mass 0.024581; collision mesh filename=package://jr_description/meshes/imu.STL; visual mesh filename=package://jr_description/meshes/imu.STL
- added link laser, mass 0.14729; collision mesh filename=package://jr_description/meshes/laser.STL; visual mesh filename=package://jr_description/meshes/laser.STL
- link arm_base: mass 0.032774 -> 0.032774128
- link base_link: mass 2.6045189845 -> 2.6045
- link front_left_wheel: mass 0.75709 -> 0.757089458454383
- link front_right_wheel: mass 0.75709 -> 0.757089458454383
- link kinect_base: mass 0.065548 -> 0.0655482560000002
Joints:
- added joint base_link_to_imu: type fixed, parent base_link, child imu, origin xyz=-0.19304 0 0.093599 rpy=0 -1.5407E-33 1.5232E-16, axis 0 0 0
- added joint base_link_to_laser: type fixed, parent base_link, child laser, origin xyz=0.03175 0 0.077724 rpy=0 -1.5407E-33 1.5232E-16, axis 0 0 0
- joint base_link_to_arm_base: origin xyz=-0.05715 0 0.0189865 rpy=0 -1.54074395550979E-33 1.52322009530389E-16 -> xyz=-0.03175 0 0.020574 rpy=0 -1.5407E-33 1.5232E-16
- joint base_link_to_front_left_wheel: origin xyz=0 0.1143 0 rpy=-1.61846129564286E-33 4.52407020283759E-18 2.46519032881566E-32 -> xyz=0 0.1143 0 rpy=-1.6185E-33 4.5241E-18 2.4652E-32
- joint base_link_to_front_right_wheel: axis 0 -1 0 -> 0 1 0
- joint base_link_to_kinect_base: origin xyz=-0.17145 0 0.157099 rpy=1.66533453693773E-16 -1.15843217122908E-16 1.0228506661306E-16 -> xyz=-0.17145 0 0.1571 rpy=1.6653E-16 -1.1584E-16 1.0229E-16
- joint base_link_to_rear_right_wheel: axis 0 -1 0 -> 0 1 0
