Commit message: Fixed joint names to append _joint

File: urdf/jr.urdf.xacro (robot description, xacro)
@@ -2,5 +2,5 @@
 <robot name="jr">
   <link name="base_footprint" />
-  <joint name="base_footprint_to_base_link" type="fixed">
+  <joint name="base_footprint_to_base_link_joint" type="fixed">
     <parent link="base_footprint" />
     <child link="base_link" />

File: urdf/jr_description.urdf (robot description, URDF)
Before this commit: robot jr_description, 9 links, 8 joints
Joints:
- removed joint base_link_to_arm_base
- removed joint base_link_to_front_left_wheel
- removed joint base_link_to_front_right_wheel
- removed joint base_link_to_imu
- removed joint base_link_to_kinect_base
- removed joint base_link_to_laser
- removed joint base_link_to_rear_left_wheel
- removed joint base_link_to_rear_right_wheel
- added joint base_link_to_arm_base_joint: type fixed, parent base_link, child arm_base, origin xyz=-0.03175 0 0.020574 rpy=0 -1.5407E-33 1.5232E-16, axis 0 0 0
- added joint base_link_to_front_left_wheel_joint: type continuous, parent base_link, child front_left_wheel, origin xyz=0 0.1143 0 rpy=-1.6185E-33 4.5241E-18 2.4652E-32, axis 0 1 0
- added joint base_link_to_front_right_wheel_joint: type continuous, parent base_link, child front_right_wheel, origin xyz=0 -0.1143 0 rpy=-4.79490768851316E-18 -2.41087784164084E-33 -2.91484050545616E-17, axis 0 1 0
- added joint base_link_to_imu_joint: type fixed, parent base_link, child imu, origin xyz=-0.19304 0 0.093599 rpy=0 -1.5407E-33 1.5232E-16, axis 0 0 0
- added joint base_link_to_kinect_base_joint: type fixed, parent base_link, child kinect_base, origin xyz=-0.17145 0 0.1571 rpy=1.6653E-16 -1.1584E-16 1.0229E-16, axis 0 0 0
- added joint base_link_to_laser_joint: type fixed, parent base_link, child laser, origin xyz=0.03175 0 0.077724 rpy=0 -1.5407E-33 1.5232E-16, axis 0 0 0
- added joint base_link_to_rear_left_wheel_joint: type continuous, parent base_link, child rear_left_wheel, origin xyz=-0.17145 0.1143 -0.00323850000000001 rpy=-5.25433558435984E-17 -1.07552855510562E-16 0, axis 0 1 0
- added joint base_link_to_rear_right_wheel_joint: type continuous, parent base_link, child rear_right_wheel, origin xyz=-0.17145 -0.1143 -0.00323849999999998 rpy=-2.84666251601602E-17 -1.66533453693773E-16 0, axis 0 1 0
